File: 4kemp.kicad_pcb (KiCad board)
At the start: 2 copper layers, 84.1 x 53 mm, 20 parts, among them SW1 SW_Push_SPDT, SW2 SW_Push_SPDT, SW3 SW_Push_SPDT, SW4 SW_Push_SPDT, SW5 RotaryEncoder_Switch, U1 102010428

Commit message: yes
Parts:
- added R1: 330o, Resistor_SMD:R_0603_1608Metric_Pad0.98x0.95mm_HandSolder, B.Cu at (56.8, 62.2)
Connections:
- D10 pad 4: unconnected-(D10-DOUT-Pad4) -> /NP2DATA
- U1 pad 8: /NPDATA -> Net-(U1-D7/CSB/P1/RX)
- U1 pad 9: /NP2DATA -> unconnected-(U1-D8/SCK/P2-Pad9)
Routing:
- net /NP2DATA: track 65.4 -> 9.40 mm, vias 2 -> 0
- net Net-(D5-A): track 14.4 -> 39.7 mm, vias 0 -> 1
- net Net-(D4-A): track 108.3 -> 87.4 mm, vias 0 -> 2
- net /Row0: track 52.5 -> 32.8 mm, vias 0 -> 2
- net +5V: track 170.4 -> 188.0 mm
- net Net-(D1-A): track 34.8 -> 46.5 mm
- net GND: track 193.0 -> 181.6 mm, vias 3 -> 2
- net Net-(LED1-DIN): track 26.6 -> 34.4 mm
- net Net-(LED3-DIN): track 33.7 -> 26.8 mm, vias 2 -> 0
- net Net-(U1-D7/CSB/P1/RX): track 0.00 -> 6.63 mm
- net /NPDATA: track 34.1 -> 29.0 mm, vias 2 -> 0
- net /A: track 39.5 -> 36.2 mm
- net Net-(D3-A): track 70.1 -> 67.3 mm
- net /Column0: track 66.9 -> 69.6 mm
- net Net-(D7-DOUT): track 28.4 -> 30.8 mm, vias 2 -> 0
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