File: 4kemp.kicad_sch (KiCad schematic)
At the start: 20 parts, among them SW1 SW_Push_SPDT, SW2 SW_Push_SPDT, SW3 SW_Push_SPDT, SW4 SW_Push_SPDT, SW5 RotaryEncoder_Switch, U1 102010428

Commit message: yes
Parts:
- added R1: 330o, Resistor_SMD:R_0603_1608Metric_Pad0.98x0.95mm_HandSolder, symbol Device:R_Small
Connections:
- net NP2DATA: now also D10.4 (DOUT); no longer U1.9 (D8/SCK/P2)
- net NPDATA: now also R1.2; no longer U1.8 (D7/CSB/P1/RX)
- new net: R1.1, U1.8 (D7/CSB/P1/RX)
Changed lines of the file:
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@@
   (no_connect (at 36.83 38.1))
   (no_connect (at 176.53 34.29))
-  (no_connect (at 93.98 88.9))
   (no_connect (at 57.15 58.42))
   (no_connect (at 176.53 44.45))
   (no_connect (at 176.53 41.91))
   (no_connect (at 36.83 58.42))
+  (no_connect (at 176.53 46.99))
   (no_connect (at 20.32 120.65))
   (no_connect (at 57.15 38.1))
@@
     (stroke (width 0) (type default))
   )
+  (wire (pts (xy 187.96 49.53) (xy 189.23 49.53))
+    (stroke (width 0) (type default))
+  )
   (wire (pts (xy 71.12 72.39) (xy 71.12 68.58))
     (stroke (width 0) (type default))
@@
     (stroke (width 0) (type default))
   )
+  (wire (pts (xy 176.53 49.53) (xy 182.88 49.53))
+    (stroke (width 0) (type default))
+  )
   (wire (pts (xy 44.45 45.72) (xy 44.45 53.34))
     (stroke (width 0) (type default))
@@
     (effects (font (size 1.27 1.27)) (justify right bottom))
   )
-  (label "NPDATA" (at 176.53 49.53 0) (fields_autoplaced)
+  (label "NP2DATA" (at 93.98 88.9 0) (fields_autoplaced)
+    (effects (font (size 1.27 1.27)) (justify left bottom))
+  )
+  (label "NPDATA" (at 189.23 49.53 0) (fields_autoplaced)
     (effects (font (size 1.27 1.27)) (justify left bottom))
   )
@@
   )
   (label "Column0" (at 26.67 20.32 0) (fields_autoplaced)
-    (effects (font (size 1.27 1.27)) (justify left bottom))
-  )
-  (label "NP2DATA" (at 176.53 46.99 0) (fields_autoplaced)
     (effects (font (size 1.27 1.27)) (justify left bottom))
   )
@@
     )
   )
+  (symbol (lib_id "Device:R_Small") (at 185.42 49.53 90) (unit 1)
+    (in_bom yes) (on_board yes) (dnp no) (fields_autoplaced)
+    (property "Reference" "R1" (at 185.42 44.45 90)
+      (effects (font (size 1.27 1.27)))
+    )
+    (property "Value" "330o" (at 185.42 46.99 90)
+      (effects (font (size 1.27 1.27)))
+    )
+    (property "Footprint" "Resistor_SMD:R_0603_1608Metric_Pad0.98x0.95mm_HandSolder" (at 185.42 49.53 0)
+      (effects (font (size 1.27 1.27)) hide)
+    )
+    (property "Datasheet" "~" (at 185.42 49.53 0)
+      (effects (font (size 1.27 1.27)) hide)
+    )
+    (pin "2")
+    (pin "1")
+    (instances
+      (project "4kemp"
+        (path "/d5595cef-bb39-4930-97fb-e1daa94dca1d"
+          (reference "R1") (unit 1)
+        )
+      )
+    )
+  )
   (symbol (lib_id "LED:SK6812") (at 25.4 88.9 0) (unit 1)
     (in_bom yes) (on_board yes) (dnp no) (fields_autoplaced)
@@
   )
   (symbol (lib_id "LED:SK6812") (at 86.36 88.9 0) (unit 1)
-    (in_bom yes) (on_board yes) (dnp no) (fields_autoplaced)
-    (property "Reference" "D10" (at 95.25 87.7921 0)
-      (effects (font (size 1.27 1.27)))
-    )
+    (in_bom yes) (on_board yes) (dnp no)
+    (property "Reference" "D10" (at 93.98 85.09 0)
+      (effects (font (size 1.27 1.27)))
+    )
